File: pcb_safe/pedal-counter.kicad_pcb (KiCad board)
At the start: 2 copper layers, 69 x 69 mm, 16 parts, among them J1 STX-3120-3B, SW1 NEW/LOAD, SW2 DEC/PREV, SW3 INC/NEXT, SW4 MODE/SAVE, SW5 OFF/ON, U1 PIICODEV_OLED_SSD1306

Commit message: <3
Parts:
- added R7: 10k, Resistor_THT:R_Axial_DIN0207_L6.3mm_D2.5mm_P10.16mm_Horizontal, B.Cu at (135.5, 54.4)
Routing:
- net +3.3V: track 77.9 -> 85.8 mm
- net 3.5MM_TRS_TIP: track 74.1 -> 81.2 mm
Other:
- board text added: "2026年8月16日 <3"
